File: Rhea - ESP32_WROOM32D.sch (KiCad schematic (older format))
At the start: 8 parts

Commit message: Power regulation updates.
Parts:
- removed D? (x2): D_ALT, symbol Device:D_ALT
- removed U?: PCF8563T, Package_SO:SOIC-8_3.9x4.9mm_P1.27mm, symbol Timer_RTC:PCF8563T
- added U2: MCP7940N-xP, symbol Timer:MCP7940N-xP
- BT1: renamed from BT?; value Battery_Cell -> BAT
- gave numbers to parts that had none: 4
Connections:
- net 3V3_SYS: now also U2.8 (VCC)
- net GNDD: now also U2.4 (VSS)
- net I2C_SCL: now also U2.6 (SCL)
- net I2C_SDA: now also U2.5 (SDA)
- net RTC_INTR: now also U2.7 (MFP)
- net at Y1.1: now also U2.1 (X1)
- net at Y1.2: now also U2.2 (X2)
- net at BT1.1 (+): now also U2.3 (VBAT)
Other:
- moved on the sheet: BT1, Y1
Changed lines of the file:
@@
 $EndSheet
 $Comp
-L Graphic:SYM_Flash_Large #SYM?
+L Graphic:SYM_Flash_Large #SYM1
 U 1 1 5E2D7EF8
 P 1725 3675
-F 0 "#SYM?" V 1575 3675 50  0001 C CNN
+F 0 "#SYM1" V 1575 3675 50  0001 C CNN
 F 1 "SYM_Flash_Large" V 1855 3675 50  0001 C CNN
 F 2 "" H 1715 3585 50  0001 C CNN
@@
 $EndSheet
 $Comp
-L Timer_RTC:PCF8563T U?
-U 1 1 5E352E79
-P 2250 6875
-F 0 "U?" H 2000 7225 50  0000 C CNN
-F 1 "PCF8563T" H 2475 7225 50  0000 C CNN
-F 2 "Package_SO:SOIC-8_3.9x4.9mm_P1.27mm" H 2250 6875 50  0001 C CNN
-F 3 "https://assets.nexperia.com/documents/data-sheet/PCF8563.pdf" H 2250 6875 50  0001 C CNN
-	1    2250 6875
-	1    0    0    -1
-$EndComp
-$Comp
-L Device:D_ALT D?
-U 1 1 5E353E7B
-P 2250 6225
-F 0 "D?" H 2325 6325 50  0000 C CNN
-F 1 "D_ALT" H 2125 6325 50  0000 C CNN
-F 2 "" H 2250 6225 50  0001 C CNN
-F 3 "~" H 2250 6225 50  0001 C CNN
-	1    2250 6225
-	0    -1   -1   0
-$EndComp
-$Comp
-L Device:D_ALT D?
-U 1 1 5E3548EE
-P 1475 6475
-F 0 "D?" H 1550 6575 50  0000 C CNN
-F 1 "D_ALT" H 1350 6575 50  0000 C CNN
-F 2 "" H 1475 6475 50  0001 C CNN
-F 3 "~" H 1475 6475 50  0001 C CNN
-	1    1475 6475
-	-1   0    0    1
-$EndComp
-$Comp
-L Device:Battery_Cell BT?
+L Device:Battery_Cell BT1
 U 1 1 5E354EF6
-P 1325 6925
-F 0 "BT?" H 1000 6975 50  0000 L CNN
-F 1 "Battery_Cell" H 825 6900 50  0000 L CNN
-F 2 "" V 1325 6985 50  0001 C CNN
-F 3 "~" V 1325 6985 50  0001 C CNN
-	1    1325 6925
-	1    0    0    -1
-$EndComp
-$Comp
-L Device:Crystal Y?
+P 1150 6675
+F 0 "BT1" H 825 6725 50  0000 L CNN
+F 1 "BAT" H 825 6650 50  0000 L CNN
+F 2 "" V 1150 6735 50  0001 C CNN
+F 3 "~" V 1150 6735 50  0001 C CNN
+	1    1150 6675
+	1    0    0    -1
+$EndComp
+$Comp
+L Device:Crystal Y1
 U 1 1 5E3556D8
-P 1800 6875
-F 0 "Y?" V 1800 6600 50  0000 L CNN
-F 1 "Crystal" V 1875 6500 50  0000 L CNN
-F 2 "" H 1800 6875 50  0001 C CNN
-F 3 "~" H 1800 6875 50  0001 C CNN
-	1    1800 6875
+P 1700 6875
+F 0 "Y1" V 1700 6600 50  0000 L CNN
+F 1 "Crystal" V 1775 6500 50  0000 L CNN
+F 2 "" H 1700 6875 50  0001 C CNN
+F 3 "~" H 1700 6875 50  0001 C CNN
+	1    1700 6875
 	0    1    1    0
 $EndComp
 Text HLabel 2775 6975 2    50   Output ~ 0
-XCLK
-Text HLabel 2775 7075 2    50   Output ~ 0
 RTC_INTR
 Wire Wire Line
-	1800 6725 1800 6675
-Wire Wire Line
-	1800 6675 1850 6675
-Wire Wire Line
-	1800 7025 1800 7075
-Wire Wire Line
-	1800 7075 1850 7075
-Wire Wire Line
-	1325 6725 1325 6475
-Wire Wire Line
-	1625 6475 2250 6475
-Wire Wire Line
 	2650 6975 2775 6975
-Wire Wire Line
-	2650 7075 2775 7075
 Wire Wire Line
 	2650 6675 3175 6675
@@
 Wire Wire Line
 	3050 5975 2250 5975
-Wire Wire Line
-	2250 5975 2250 6075
-Wire Wire Line
-	2250 6375 2250 6475
-Connection ~ 2250 6475
 Text Label 3050 5975 2    50   ~ 0
 3V3_SYS
@@
 	3450 5650 675  5650
 $Comp
-L power:GNDD #PWR0101
+L power:GNDD #PWR06
 U 1 1 5E3860B8
-P 1325 7025
-F 0 "#PWR0101" H 1325 6775 50  0001 C CNN
-F 1 "GNDD" H 1329 6870 50  0000 C CNN
-F 2 "" H 1325 7025 50  0001 C CNN
-F 3 "" H 1325 7025 50  0001 C CNN
-	1    1325 7025
-	1    0    0    -1
-$EndComp
-$Comp
-L power:GNDD #PWR0102
+P 1150 6775
+F 0 "#PWR06" H 1150 6525 50  0001 C CNN
+F 1 "GNDD" H 1154 6620 50  0000 C CNN
+F 2 "" H 1150 6775 50  0001 C CNN
+F 3 "" H 1150 6775 50  0001 C CNN
+	1    1150 6775
+	1    0    0    -1
+$EndComp
+$Comp
+L power:GNDD #PWR09
 U 1 1 5E386591
 P 2250 7275
-F 0 "#PWR0102" H 2250 7025 50  0001 C CNN
+F 0 "#PWR09" H 2250 7025 50  0001 C CNN
 F 1 "GNDD" H 2254 7120 50  0000 C CNN
 F 2 "" H 2250 7275 50  0001 C CNN
@@
 $EndComp
 $Comp
-L Connector:Micro_SD_Card J?
+L Connector:Micro_SD_Card J1
 U 1 1 5E2A33C5
 P 5700 6625
-F 0 "J?" H 5650 7342 50  0000 C CNN
+F 0 "J1" H 5650 7342 50  0000 C CNN
 F 1 "Micro_SD_Card" H 5650 7251 50  0000 C CNN
 F 2 "" H 6850 6925 50  0001 C CNN
@@
 NoConn ~ 4800 7025
 $Comp
-L BME280:TEMP-HUM-PRES-BME280 U?
+L BME280:TEMP-HUM-PRES-BME280 U1
 U 1 1 5E2B157D
 P 8475 1875
-F 0 "U?" H 8425 1500 50  0000 L CNN
+F 0 "U1" H 8425 1500 50  0000 L CNN
 F 1 "TEMP-HUM-PRES-BME280" H 7950 2350 50  0000 L CNN
 F 2 "TEMP-HUM-PRES-BME280" H 8475 1875 50  0001 L BNN
@@
 	4250 6925 4800 6925
 $Comp
-L power:GNDD #PWR0103
+L power:GNDD #PWR07
 U 1 1 5E2C2546
 P 4700 7225
-F 0 "#PWR0103" H 4700 6975 50  0001 C CNN
+F 0 "#PWR07" H 4700 6975 50  0001 C CNN
 F 1 "GNDD" H 4704 7070 50  0000 C CNN
 F 2 "" H 4700 7225 50  0001 C CNN
@@
 	6600 5650 3825 5650
 $Comp
-L power:Earth #PWR0105
+L power:Earth #PWR08
 U 1 1 5E2D1368
 P 6500 7225
-F 0 "#PWR0105" H 6500 6975 50  0001 C CNN
+F 0 "#PWR08" H 6500 6975 50  0001 C CNN
 F 1 "Earth" H 6500 7075 50  0001 C CNN
 F 2 "" H 6500 7225 50  0001 C CNN
@@
 $EndComp
 $Comp
-L power:GNDD #PWR0108
+L power:GNDD #PWR05
 U 1 1 5E30527C
 P 9225 2100
-F 0 "#PWR0108" H 9225 1850 50  0001 C CNN
+F 0 "#PWR05" H 9225 1850 50  0001 C CNN
 F 1 "GNDD" H 9229 1945 50  0000 C CNN
 F 2 "" H 9225 2100 50  0001 C CNN
@@
 	4150 3550 4975 3550
 $Comp
-L Device:Net-Tie_4 NT?
+L Device:Net-Tie_4 NT1
 U 1 1 5E3B6F89
 P 6925 1600
-F 0 "NT?" H 6925 1781 50  0000 C CNN
+F 0 "NT1" H 6925 1781 50  0000 C CNN
 F 1 "Net-Tie_4" H 6925 1690 50  0000 C CNN
 F 2 "" H 6925 1600 50  0001 C CNN
@@
 $EndComp
 $Comp
-L power:GNDA #PWR0109
+L power:GNDA #PWR02
 U 1 1 5E3B876E
 P 6775 1725
-F 0 "#PWR0109" H 6775 1475 50  0001 C CNN
+F 0 "#PWR02" H 6775 1475 50  0001 C CNN
 F 1 "GNDA" H 6775 1575 50  0000 C CNN
 F 2 "" H 6775 1725 50  0001 C CNN
@@
 $EndComp
 $Comp
-L power:GNDD #PWR0110
+L power:GNDD #PWR03
 U 1 1 5E3B8EA3
 P 7075 1725
-F 0 "#PWR0110" H 7075 1475 50  0001 C CNN
+F 0 "#PWR03" H 7075 1475 50  0001 C CNN
 F 1 "GNDD" H 7075 1575 50  0000 C CNN
 F 2 "" H 7075 1725 50  0001 C CNN
@@
 	7075 1700 7075 1725
 $Comp
-L power:GNDPWR #PWR0111
+L power:GNDPWR #PWR04
 U 1 1 5E3BC318
 P 7375 1725
-F 0 "#PWR0111" H 7375 1525 50  0001 C CNN
+F 0 "#PWR04" H 7375 1525 50  0001 C CNN
 F 1 "GNDPWR" H 7375 1575 50  0000 C CNN
 F 2 "" H 7375 1675 50  0001 C CNN
@@
 Grounds
 $Comp
-L power:Earth_Protective #PWR?
+L power:Earth_Protective #PWR01
 U 1 1 5E63B8FE
 P 6525 1725
-F 0 "#PWR?" H 6775 1475 50  0001 C CNN
+F 0 "#PWR01" H 6775 1475 50  0001 C CNN
 F 1 "Earth_Protective" H 6975 1575 50  0001 C CNN
 F 2 "" H 6525 1625 50  0001 C CNN
@@
 Wire Bus Line
 	2425 3675 5100 3675
+$Comp
+L Timer:MCP7940N-xP U2
+U 1 1 5E440421
+P 2250 6875
+F 0 "U2" H 2500 7250 50  0000 C CNN
+F 1 "MCP7940N-xP" H 1925 7250 50  0000 C CNN
+F 2 "" H 2250 6875 50  0001 C CNN
+F 3 "http://ww1.microchip.com/downloads/en/DeviceDoc/20005010F.pdf" H 2250 6875 50  0001 C CNN
+	1    2250 6875
+	-1   0    0    -1
+$EndComp
+Wire Wire Line
+	1150 6450 2150 6450
+Wire Wire Line
+	2250 5975 2250 6475
+Wire Wire Line
+	1700 7025 1850 7025
+Wire Wire Line
+	1850 7025 1850 6975
+Wire Wire Line
+	1700 6725 1850 6725
+Wire Wire Line
+	1850 6725 1850 6775
+Wire Wire Line
+	1150 6450 1150 6475
+Wire Wire Line
+	2150 6450 2150 6475
 Wire Bus Line
 	9700 1975 9700 3425
