File: ext_headers.sch (KiCad schematic (older format))
At the start: 0 parts

Commit message: External headers early draft.
Parts:
- added J?: Conn_02x08_Counter_Clockwise, symbol Connector_Generic:Conn_02x08_Counter_Clockwise
- added J? (x2): Conn_01x08, symbol Connector_Generic:Conn_01x08
- added J?: Conn_02x03_Counter_Clockwise, symbol Connector_Generic:Conn_02x03_Counter_Clockwise
- added R? (x32): 200R, symbol Device:R_US
- added U? (x4): NUF8402MN, Package_DFN_QFN:DFN-16-1EP_3x5mm_P0.5mm_EP1.66x4.4mm, symbol Power_Protection:NUF8402MN
- added U?: TCA9555DBR, Package_SO:SSOP-24_5.3x8.2mm_P0.65mm, symbol Interface_Expansion:TCA9555DBR
Connections:
- new net: J?.1 (Pin_1), R?.1 (x2)
- new net: J?.2 (Pin_2), R?.1 (x2)
- new net: J?.3 (Pin_3), R?.1 (x2)
- new net: J?.4 (Pin_4), R?.1 (x2)
- new net: J?.5 (Pin_5), R?.1 (x2)
- new net: J?.6 (Pin_6), R?.1 (x2)
- new net: J?.7 (Pin_7), R?.1 (x2)
- new net: J?.8 (Pin_8), R?.1 (x2)
- new net: R?.2, U?.10 (Ch7_Out) (x4)
- new net: R?.2, U?.11 (Ch6_Out) (x4)
- new net: R?.2, U?.12 (Ch5_Out) (x4)
- new net: R?.2, U?.13 (Ch4_Out) (x4)
- new net: R?.2, U?.14 (Ch3_Out) (x4)
- new net: R?.2, U?.15 (Ch2_Out) (x4)
- new net: R?.2, U?.16 (Ch1_Out) (x4)
- new net: R?.2, U?.9 (Ch8_Out) (x4)
- new net: U?.1 (Ch1_In), U?.4 (P00)
- new net: U?.2 (Ch2_In), U?.5 (P01)
- new net: U?.3 (Ch3_In), U?.6 (P02)
- new net: U?.4 (Ch4_In), U?.7 (P03)
- new net: U?.5 (Ch5_In), U?.8 (P04)
- new net: U?.6 (Ch6_In), U?.9 (P05)
- new net: U?.10 (P06), U?.7 (Ch7_In)
- new net: U?.11 (P07), U?.8 (Ch8_In)
- new net: U?.1 (Ch1_In), U?.13 (P10)
- new net: U?.14 (P11), U?.2 (Ch2_In)
- new net: U?.15 (P12), U?.3 (Ch3_In)
- new net: U?.16 (P13), U?.4 (Ch4_In)
- new net: U?.17 (P14), U?.5 (Ch5_In)
- new net: U?.18 (P15), U?.6 (Ch6_In)
- new net: U?.19 (P16), U?.7 (Ch7_In)
- new net: U?.20 (P17), U?.8 (Ch8_In)
- new net 3V3_EXT: J?.6 (Pin_6)
- new net 3V3_SYS: J?.5 (Pin_5)
- new net ADIO0: U?.1 (Ch1_In)
- new net ADIO1: U?.2 (Ch2_In)
- new net ADIO2: U?.3 (Ch3_In)
- new net ADIO3: U?.4 (Ch4_In)
- new net ADIO4: U?.5 (Ch5_In)
- new net ADIO5: U?.6 (Ch6_In)
- new net ADIO6: U?.7 (Ch7_In)
- new net ADIO7: U?.8 (Ch8_In)
- new net CAN_RX: U?.6 (Ch6_In)
- new net CAN_TX: U?.7 (Ch7_In)
- new net D0: J?.1 (Pin_1), R?.1
- new net D1: J?.2 (Pin_2), R?.1
- new net D10: J?.11 (Pin_11), R?.1
- new net D11: J?.12 (Pin_12), R?.1
- new net D12: J?.13 (Pin_13), R?.1
- new net D13: J?.14 (Pin_14), R?.1
- new net D14: J?.15 (Pin_15), R?.1
- new net D15: J?.16 (Pin_16), R?.1
- new net D2: J?.3 (Pin_3), R?.1
- new net D3: J?.4 (Pin_4), R?.1
- new net D4: J?.5 (Pin_5), R?.1
- new net D5: J?.6 (Pin_6), R?.1
- new net D6: J?.7 (Pin_7), R?.1
- new net D7: J?.8 (Pin_8), R?.1
- new net D8: J?.9 (Pin_9), R?.1
- new net D9: J?.10 (Pin_10), R?.1
- new net DIO_INTR: U?.1 (~INT)
- new net Earth_Protective: J?.3 (Pin_3), U?.17 (GND), U?.17 (GND), U?.17 (GND), U?.17 (GND)
- new net GNDA: J?.1 (Pin_1)
- new net GNDD: J?.2 (Pin_2), U?.12 (GND)
- new net I2C_SCL: U?.1 (Ch1_In), U?.22 (SCL)
- new net I2C_SDA: U?.2 (Ch2_In), U?.23 (SDA)
- new net SPI_CLK: U?.5 (Ch5_In)
- new net SPI_MISO: U?.3 (Ch3_In)
- new net SPI_MOSI: U?.4 (Ch4_In)
- new net XCLK: U?.8 (Ch8_In)
- new net ~RESET: J?.4 (Pin_4)
Other:
- note added: "A/D General Purpose IO"
- note added: "Application notes:"
- note added: "Bus Communication Lines"
- note added: "Digital IO Expansion"
- note added: "JTAG???"
- note added: "PCAL6416A???"
- note added: "Power & Control Signals"

Commit message: Power regulation updates.
Parts:
- gave numbers to parts that had none: 41
